File: hardware/kicad/esphome-sensor.kicad_sch (KiCad schematic)
At the start: 26 parts, among them J1 DC POWER IN, J2 OLED, J3 1WIRE-BUS1, J4 1WIRE-BUS2, J5 I2C, U1 D24V5F5, U2 FeatherS3D

Commit message: filter cap defined
Parts:
- C1: value C_Polarized -> 100uF 35V
Changed lines of the file:
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@@
 			)
 		)
-		(property "Value" "C_Polarized"
+		(property "Value" "100uF 35V"
 			(at 54.61 42.2909 0)
 			(effects
